File: ICED - Left/ICEDLeft.kicad_sch (KiCad schematic)
At the start: 76 parts

Commit message: Left: Revert to SMD diodes
Parts:
- D1, D10, D11, D12, D13, D14, D15, D16, D17, D18, D19, D2, D20, D21, D22, D23, D24, D25, D26, D27, D28, D29, D3, D30, D31, D32, D33, D34, D35, D36, D37, D38, D4, D5, D6, D7, D8, D9: footprint prettylib:1N4148 -> prettylib:SOT123-DIODE
